File: Kairos.sch (KiCad schematic (older format))
At the start: 40 parts, among them J1 USB_mini_micro_B, Q1 NSS40301MZ4T1G, SW1 SW_RST1, U1 ATMEGA32U2-AU, Y1 Crystal

Commit message: Fix left shift, associate MX footprints
Parts:
- Q1: footprint TO_SOT_Packages_SMD:SOT-223 -> (none)
- U1: footprint TQFP-32 -> (none)
Changed lines of the file:
@@
 F 0 "U1" H 2200 4400 50  0000 C CNN
 F 1 "ATMEGA32U2-AU" H 3800 1700 50  0000 C CNN
-F 2 "TQFP-32" H 2900 3100 50  0001 C CNN
+F 2 "" H 2900 3100 50  0001 C CNN
 F 3 "http://www.atmel.com/Images/doc7799.pdf" H 3150 1600 50  0001 C CNN
 	1    3050 3050
@@
 F 0 "Q1" H 4150 1275 50  0000 L CNN
 F 1 "NSS40301MZ4T1G" H 4150 1200 50  0000 L CNN
-F 2 "TO_SOT_Packages_SMD:SOT-223" H 4150 1125 50  0001 L CIN
+F 2 "" H 4150 1125 50  0001 L CIN
 F 3 "" H 3950 1200 50  0001 L CNN
 	1    3950 1200
@@
 F 0 "LED1" H 9050 800 60  0000 C CNN
 F 1 "WS2812B" H 9050 1600 60  0000 C CNN
-F 2 "" V 9000 1200 60  0000 C CNN
+F 2 "" V 9000 1200 60  0001 C CNN
 F 3 "" V 9000 1200 60  0000 C CNN
 	1    9050 1200
@@
 F 0 "LED2" H 9050 1750 60  0000 C CNN
 F 1 "WS2812B" H 9050 2550 60  0000 C CNN
-F 2 "" V 9000 2150 60  0000 C CNN
+F 2 "" V 9000 2150 60  0001 C CNN
 F 3 "" V 9000 2150 60  0000 C CNN
 	1    9050 2150
@@
 F 0 "LED3" H 9050 2700 60  0000 C CNN
 F 1 "WS2812B" H 9050 3500 60  0000 C CNN
-F 2 "" V 9000 3100 60  0000 C CNN
+F 2 "" V 9000 3100 60  0001 C CNN
 F 3 "" V 9000 3100 60  0000 C CNN
 	1    9050 3100
@@
 F 0 "LED4" H 9050 3650 60  0000 C CNN
 F 1 "WS2812B" H 9050 4450 60  0000 C CNN
-F 2 "" V 9000 4050 60  0000 C CNN
+F 2 "" V 9000 4050 60  0001 C CNN
 F 3 "" V 9000 4050 60  0000 C CNN
 	1    9050 4050
@@
 F 0 "LED5" H 9050 4600 60  0000 C CNN
 F 1 "WS2812B" H 9050 5400 60  0000 C CNN
-F 2 "" V 9000 5000 60  0000 C CNN
+F 2 "" V 9000 5000 60  0001 C CNN
 F 3 "" V 9000 5000 60  0000 C CNN
 	1    9050 5000
@@
 F 0 "LED6" H 9050 5550 60  0000 C CNN
 F 1 "WS2812B" H 9050 6350 60  0000 C CNN
-F 2 "" V 9000 5950 60  0000 C CNN
+F 2 "" V 9000 5950 60  0001 C CNN
 F 3 "" V 9000 5950 60  0000 C CNN
 	1    9050 5950
@@
 F 0 "LED7" H 10500 800 60  0000 C CNN
 F 1 "WS2812B" H 10500 1600 60  0000 C CNN
-F 2 "" V 10450 1200 60  0000 C CNN
+F 2 "" V 10450 1200 60  0001 C CNN
 F 3 "" V 10450 1200 60  0000 C CNN
 	1    10500 1200
@@
 F 0 "LED8" H 10500 1750 60  0000 C CNN
 F 1 "WS2812B" H 10500 2550 60  0000 C CNN
-F 2 "" V 10450 2150 60  0000 C CNN
+F 2 "" V 10450 2150 60  0001 C CNN
 F 3 "" V 10450 2150 60  0000 C CNN
 	1    10500 2150
@@
 F 0 "LED9" H 10500 2700 60  0000 C CNN
 F 1 "WS2812B" H 10500 3500 60  0000 C CNN
-F 2 "" V 10450 3100 60  0000 C CNN
+F 2 "" V 10450 3100 60  0001 C CNN
 F 3 "" V 10450 3100 60  0000 C CNN
 	1    10500 3100
@@
 F 0 "LED10" H 10500 3650 60  0000 C CNN
 F 1 "WS2812B" H 10500 4450 60  0000 C CNN
-F 2 "" V 10450 4050 60  0000 C CNN
+F 2 "" V 10450 4050 60  0001 C CNN
 F 3 "" V 10450 4050 60  0000 C CNN
 	1    10500 4050
@@
 F 0 "LED11" H 10500 4600 60  0000 C CNN
 F 1 "WS2812B" H 10500 5400 60  0000 C CNN
-F 2 "" V 10450 5000 60  0000 C CNN
+F 2 "" V 10450 5000 60  0001 C CNN
 F 3 "" V 10450 5000 60  0000 C CNN
 	1    10500 5000
@@
 F 0 "LED12" H 10500 5550 60  0000 C CNN
 F 1 "WS2812B" H 10500 6350 60  0000 C CNN
-F 2 "" V 10450 5950 60  0000 C CNN
+F 2 "" V 10450 5950 60  0001 C CNN
 F 3 "" V 10450 5950 60  0000 C CNN
 	1    10500 5950
@@
 F 0 "SW1" H 1750 2260 50  0000 C CNN
 F 1 "SW_RST1" H 1600 2070 50  0000 C CNN
-F 2 "" H 1600 2150 60  0000 C CNN
+F 2 "" H 1600 2150 60  0001 C CNN
 F 3 "" H 1600 2150 60  0000 C CNN
 	1    1600 2150
@@
 F 0 "J1" H 600 4400 60  0000 C CNN
 F 1 "USB_mini_micro_B" H 850 4700 60  0001 C CNN
-F 2 "" H 950 4450 60  0000 C CNN
+F 2 "" H 950 4450 60  0001 C CNN
 F 3 "" H 950 4450 60  0000 C CNN
 	1    1000 4450
