File: rightmods.sch (KiCad schematic (older format))
At the start: 0 parts

Commit message: Some edits
Other:
- note added: "1"
- note added: "No Clue"
- note added: "Right Mods\n"
Changed lines of the file:
@@
 $Descr A4 11693 8268
 encoding utf-8
-Sheet 1 7
+Sheet 5 7
 Title ""
 Date ""
@@
 Comment4 ""
 $EndDescr
+Text Notes 7325 7500 0    60   ~ 0
+Right Mods\n
+Text Notes 8100 7650 0    60   ~ 0
+No Clue
+Text Notes 10550 7650 0    60   ~ 0
+1
 $EndSCHEMATC

Commit message: Added right mods
Parts:
- added DRM1, DRM2, DRM3, DRM4, DRM5: 1N4148WS, symbol D
- added RM1, RM11, RM3, RM7, RM8, RM9: MX-1U, symbol MX-1U
- added RM10, RM2, RM4, RM6: MX-1.25U, symbol MX-1.25U
- added RM12, RM5: MX-1.5U, symbol MX-1.5U
- added RRM1, RRM2, RRM3, RRM4, RRM5: 2.2k, symbol R
Connections:
- new net: DRM1.1 (K), RM1.1 (COL), RM2.1 (COL)
- new net: RM1.3 (LED), RM2.3 (LED), RRM1.1
- new net: DRM2.1 (K), RM3.1 (COL), RM4.1 (COL), RM5.1 (COL)
- new net: RM3.3 (LED), RM4.3 (LED), RM5.3 (LED), RRM2.1
- new net: DRM4.1 (K), RM6.1 (COL), RM7.1 (COL), RM9.1 (COL)
- new net: RM6.3 (LED), RM7.3 (LED), RM9.3 (LED), RRM4.1
- new net: DRM3.1 (K), RM8.1 (COL)
- new net: RM8.3 (LED), RRM3.1
- new net: DRM5.1 (K), RM10.1 (COL), RM11.1 (COL), RM12.1 (COL)
- new net: RM10.3 (LED), RM11.3 (LED), RM12.3 (LED), RRM5.1
- new net rightmods5V: RRM1.2, RRM2.2, RRM3.2, RRM4.2, RRM5.2
- new net rightmodsLEDGND: RM1.4 (LEDGND), RM10.4 (LEDGND), RM11.4 (LEDGND), RM12.4 (LEDGND), RM2.4 (LEDGND), RM3.4 (LEDGND), RM4.4 (LEDGND), RM5.4 (LEDGND), RM6.4 (LEDGND), RM7.4 (LEDGND), RM8.4 (LEDGND), RM9.4 (LEDGND)
- new net rightmodscol1: DRM1.2 (A)
- new net rightmodscol2: DRM2.2 (A), DRM3.2 (A)
- new net rightmodscol3: DRM4.2 (A), DRM5.2 (A)
- new net rightmodsrow1: RM3.2 (ROW), RM4.2 (ROW), RM5.2 (ROW), RM6.2 (ROW), RM7.2 (ROW), RM9.2 (ROW)
- new net rightmodsrow2: RM1.2 (ROW), RM10.2 (ROW), RM11.2 (ROW), RM12.2 (ROW), RM2.2 (ROW), RM8.2 (ROW)

Commit message: Fix all key annotations
Parts:
- renumbered RM1 to K_RM1, RM10 to K_RM10, RM11 to K_RM11, RM12 to K_RM12, RM2 to K_RM2, RM3 to K_RM3, RM4 to K_RM4, RM5 to K_RM5, RM6 to K_RM6, RM7 to K_RM7, RM8 to K_RM8, RM9 to K_RM9
Changed lines of the file:
@@
 1
 $Comp
-L MX-1U RM1
+L MX-1U K_RM1
 U 1 1 5930D685
 P 4125 2700
-F 0 "RM1" H 4125 2825 60  0000 C CNN
+F 0 "K_RM1" H 4125 2825 60  0000 C CNN
 F 1 "MX-1U" H 4125 2750 20  0000 C CNN
 F 2 "" H 4100 2675 60  0001 C CNN
@@
 $EndComp
 $Comp
-L MX-1.25U RM2
+L MX-1.25U K_RM2
 U 1 1 5930D6AD
 P 4125 3275
-F 0 "RM2" H 4125 3400 60  0000 C CNN
+F 0 "K_RM2" H 4125 3400 60  0000 C CNN
 F 1 "MX-1.25U" H 4125 3325 20  0000 C CNN
 F 2 "" H 4100 3250 60  0001 C CNN
@@
 $EndComp
 $Comp
-L MX-1U RM3
+L MX-1U K_RM3
 U 1 1 5930D721
 P 4525 2700
-F 0 "RM3" H 4525 2825 60  0000 C CNN
+F 0 "K_RM3" H 4525 2825 60  0000 C CNN
 F 1 "MX-1U" H 4525 2750 20  0000 C CNN
 F 2 "" H 4500 2675 60  0001 C CNN
@@
 $EndComp
 $Comp
-L MX-1.25U RM4
+L MX-1.25U K_RM4
 U 1 1 5930D74B
 P 4525 3275
-F 0 "RM4" H 4525 3400 60  0000 C CNN
+F 0 "K_RM4" H 4525 3400 60  0000 C CNN
 F 1 "MX-1.25U" H 4525 3325 20  0000 C CNN
 F 2 "" H 4500 3250 60  0001 C CNN
@@
 $EndComp
 $Comp
-L MX-1.5U RM5
+L MX-1.5U K_RM5
 U 1 1 5930D77D
 P 4525 3850
-F 0 "RM5" H 4525 3975 60  0000 C CNN
+F 0 "K_RM5" H 4525 3975 60  0000 C CNN
 F 1 "MX-1.5U" H 4525 3900 20  0000 C CNN
 F 2 "" H 4500 3825 60  0001 C CNN
@@
 $EndComp
 $Comp
-L MX-1.25U RM6
+L MX-1.25U K_RM6
 U 1 1 5930DAAE
 P 5325 3275
-F 0 "RM6" H 5325 3400 60  0000 C CNN
+F 0 "K_RM6" H 5325 3400 60  0000 C CNN
 F 1 "MX-1.25U" H 5325 3325 20  0000 C CNN
 F 2 "" H 5300 3250 60  0001 C CNN
@@
 $EndComp
 $Comp
-L MX-1U RM7
+L MX-1U K_RM7
 U 1 1 5930DAF4
 P 5325 3850
-F 0 "RM7" H 5325 3975 60  0000 C CNN
+F 0 "K_RM7" H 5325 3975 60  0000 C CNN
 F 1 "MX-1U" H 5325 3900 20  0000 C CNN
 F 2 "" H 5300 3825 60  0001 C CNN
@@
 $EndComp
 $Comp
-L MX-1U RM8
+L MX-1U K_RM8
 U 1 1 5930DB99
 P 4925 2700
-F 0 "RM8" H 4925 2825 60  0000 C CNN
+F 0 "K_RM8" H 4925 2825 60  0000 C CNN
 F 1 "MX-1U" H 4925 2750 20  0000 C CNN
 F 2 "" H 4900 2675 60  0001 C CNN
@@
 $EndComp
 $Comp
-L MX-1U RM9
+L MX-1U K_RM9
 U 1 1 5930DBD5
 P 5325 2700
-F 0 "RM9" H 5325 2825 60  0000 C CNN
+F 0 "K_RM9" H 5325 2825 60  0000 C CNN
 F 1 "MX-1U" H 5325 2750 20  0000 C CNN
 F 2 "" H 5300 2675 60  0001 C CNN
@@
 $EndComp
 $Comp
-L MX-1.25U RM10
+L MX-1.25U K_RM10
 U 1 1 5930DD71
 P 5725 3275
-F 0 "RM10" H 5725 3400 60  0000 C CNN
+F 0 "K_RM10" H 5725 3400 60  0000 C CNN
 F 1 "MX-1.25U" H 5725 3325 20  0000 C CNN
 F 2 "" H 5700 3250 60  0001 C CNN
@@
 $EndComp
 $Comp
-L MX-1U RM11
+L MX-1U K_RM11
 U 1 1 5930DDB5
 P 5725 2700
-F 0 "RM11" H 5725 2825 60  0000 C CNN
+F 0 "K_RM11" H 5725 2825 60  0000 C CNN
 F 1 "MX-1U" H 5725 2750 20  0000 C CNN
 F 2 "" H 5700 2675 60  0001 C CNN
@@
 $EndComp
 $Comp
-L MX-1.5U RM12
+L MX-1.5U K_RM12
 U 1 1 5930DF10
 P 5725 3850
-F 0 "RM12" H 5725 3975 60  0000 C CNN
+F 0 "K_RM12" H 5725 3975 60  0000 C CNN
 F 1 "MX-1.5U" H 5725 3900 20  0000 C CNN
 F 2 "" H 5700 3825 60  0001 C CNN

Commit message: Fix left shift, associate MX footprints
Parts:
- K_RM1, K_RM11, K_RM3, K_RM7, K_RM8, K_RM9: footprint (none) -> MX_Alps_Hybrid:MX-1U
- K_RM10, K_RM2, K_RM4, K_RM6: footprint (none) -> MX_Alps_Hybrid:MX-1.25U
- K_RM12, K_RM5: footprint (none) -> MX_Alps_Hybrid:MX-1.5U
Changed lines of the file:
@@
 F 0 "K_RM1" H 4125 2825 60  0000 C CNN
 F 1 "MX-1U" H 4125 2750 20  0000 C CNN
-F 2 "" H 4100 2675 60  0001 C CNN
+F 2 "MX_Alps_Hybrid:MX-1U" H 4100 2675 60  0001 C CNN
 F 3 "" H 4100 2675 60  0001 C CNN
 	1    4125 2700
@@
 F 0 "K_RM2" H 4125 3400 60  0000 C CNN
 F 1 "MX-1.25U" H 4125 3325 20  0000 C CNN
-F 2 "" H 4100 3250 60  0001 C CNN
+F 2 "MX_Alps_Hybrid:MX-1.25U" H 4100 3250 60  0001 C CNN
 F 3 "" H 4100 3250 60  0001 C CNN
 	1    4125 3275
@@
 F 0 "K_RM3" H 4525 2825 60  0000 C CNN
 F 1 "MX-1U" H 4525 2750 20  0000 C CNN
-F 2 "" H 4500 2675 60  0001 C CNN
+F 2 "MX_Alps_Hybrid:MX-1U" H 4500 2675 60  0001 C CNN
 F 3 "" H 4500 2675 60  0001 C CNN
 	1    4525 2700
@@
 F 0 "K_RM4" H 4525 3400 60  0000 C CNN
 F 1 "MX-1.25U" H 4525 3325 20  0000 C CNN
-F 2 "" H 4500 3250 60  0001 C CNN
+F 2 "MX_Alps_Hybrid:MX-1.25U" H 4500 3250 60  0001 C CNN
 F 3 "" H 4500 3250 60  0001 C CNN
 	1    4525 3275
@@
 F 0 "K_RM5" H 4525 3975 60  0000 C CNN
 F 1 "MX-1.5U" H 4525 3900 20  0000 C CNN
-F 2 "" H 4500 3825 60  0001 C CNN
+F 2 "MX_Alps_Hybrid:MX-1.5U" H 4500 3825 60  0001 C CNN
 F 3 "" H 4500 3825 60  0001 C CNN
 	1    4525 3850
@@
 F 0 "K_RM6" H 5325 3400 60  0000 C CNN
 F 1 "MX-1.25U" H 5325 3325 20  0000 C CNN
-F 2 "" H 5300 3250 60  0001 C CNN
+F 2 "MX_Alps_Hybrid:MX-1.25U" H 5300 3250 60  0001 C CNN
 F 3 "" H 5300 3250 60  0001 C CNN
 	1    5325 3275
@@
 F 0 "K_RM7" H 5325 3975 60  0000 C CNN
 F 1 "MX-1U" H 5325 3900 20  0000 C CNN
-F 2 "" H 5300 3825 60  0001 C CNN
+F 2 "MX_Alps_Hybrid:MX-1U" H 5300 3825 60  0001 C CNN
 F 3 "" H 5300 3825 60  0001 C CNN
 	1    5325 3850
@@
 F 0 "K_RM8" H 4925 2825 60  0000 C CNN
 F 1 "MX-1U" H 4925 2750 20  0000 C CNN
-F 2 "" H 4900 2675 60  0001 C CNN
+F 2 "MX_Alps_Hybrid:MX-1U" H 4900 2675 60  0001 C CNN
 F 3 "" H 4900 2675 60  0001 C CNN
 	1    4925 2700
@@
 F 0 "K_RM9" H 5325 2825 60  0000 C CNN
 F 1 "MX-1U" H 5325 2750 20  0000 C CNN
-F 2 "" H 5300 2675 60  0001 C CNN
+F 2 "MX_Alps_Hybrid:MX-1U" H 5300 2675 60  0001 C CNN
 F 3 "" H 5300 2675 60  0001 C CNN
 	1    5325 2700
@@
 F 0 "K_RM10" H 5725 3400 60  0000 C CNN
 F 1 "MX-1.25U" H 5725 3325 20  0000 C CNN
-F 2 "" H 5700 3250 60  0001 C CNN
+F 2 "MX_Alps_Hybrid:MX-1.25U" H 5700 3250 60  0001 C CNN
 F 3 "" H 5700 3250 60  0001 C CNN
 	1    5725 3275
@@
 F 0 "K_RM11" H 5725 2825 60  0000 C CNN
 F 1 "MX-1U" H 5725 2750 20  0000 C CNN
-F 2 "" H 5700 2675 60  0001 C CNN
+F 2 "MX_Alps_Hybrid:MX-1U" H 5700 2675 60  0001 C CNN
 F 3 "" H 5700 2675 60  0001 C CNN
 	1    5725 2700
@@
 F 0 "K_RM12" H 5725 3975 60  0000 C CNN
 F 1 "MX-1.5U" H 5725 3900 20  0000 C CNN
-F 2 "" H 5700 3825 60  0001 C CNN
+F 2 "MX_Alps_Hybrid:MX-1.5U" H 5700 3825 60  0001 C CNN
 F 3 "" H 5700 3825 60  0001 C CNN
 	1    5725 3850
@@
 F 0 "DRM1" H 4375 2400 50  0000 C CNN
 F 1 "1N4148WS" H 4375 2200 50  0000 C CNN
-F 2 "" H 4375 2300 50  0000 C CNN
+F 2 "" H 4375 2300 50  0001 C CNN
 F 3 "" H 4375 2300 50  0000 C CNN
 	1    4375 2300
@@
 F 0 "DRM2" H 4775 2400 50  0000 C CNN
 F 1 "1N4148WS" H 4775 2200 50  0000 C CNN
-F 2 "" H 4775 2300 50  0000 C CNN
+F 2 "" H 4775 2300 50  0001 C CNN
 F 3 "" H 4775 2300 50  0000 C CNN
 	1    4775 2300
@@
 F 0 "DRM3" H 5175 2400 50  0000 C CNN
 F 1 "1N4148WS" H 5175 2200 50  0000 C CNN
-F 2 "" H 5175 2300 50  0000 C CNN
+F 2 "" H 5175 2300 50  0001 C CNN
 F 3 "" H 5175 2300 50  0000 C CNN
 	1    5175 2300
@@
 F 0 "DRM4" H 5575 2400 50  0000 C CNN
 F 1 "1N4148WS" H 5575 2200 50  0000 C CNN
-F 2 "" H 5575 2300 50  0000 C CNN
+F 2 "" H 5575 2300 50  0001 C CNN
 F 3 "" H 5575 2300 50  0000 C CNN
 	1    5575 2300
@@
 F 0 "DRM5" H 5975 2400 50  0000 C CNN
 F 1 "1N4148WS" H 5975 2200 50  0000 C CNN
-F 2 "" H 5975 2300 50  0000 C CNN
+F 2 "" H 5975 2300 50  0001 C CNN
 F 3 "" H 5975 2300 50  0000 C CNN
 	1    5975 2300
@@
 F 0 "RRM1" V 4480 4525 50  0000 C CNN
 F 1 "2.2k" V 4400 4525 50  0000 C CNN
-F 2 "" V 4330 4525 50  0000 C CNN
+F 2 "" V 4330 4525 50  0001 C CNN
 F 3 "" H 4400 4525 50  0000 C CNN
 	1    4400 4525
@@
 F 0 "RRM2" V 4880 4525 50  0000 C CNN
 F 1 "2.2k" V 4800 4525 50  0000 C CNN
-F 2 "" V 4730 4525 50  0000 C CNN
+F 2 "" V 4730 4525 50  0001 C CNN
 F 3 "" H 4800 4525 50  0000 C CNN
 	1    4800 4525
@@
 F 0 "RRM3" V 5280 4525 50  0000 C CNN
 F 1 "2.2k" V 5200 4525 50  0000 C CNN
-F 2 "" V 5130 4525 50  0000 C CNN
+F 2 "" V 5130 4525 50  0001 C CNN
 F 3 "" H 5200 4525 50  0000 C CNN
 	1    5200 4525
@@
 F 0 "RRM4" V 5680 4525 50  0000 C CNN
 F 1 "2.2k" V 5600 4525 50  0000 C CNN
-F 2 "" V 5530 4525 50  0000 C CNN
+F 2 "" V 5530 4525 50  0001 C CNN
 F 3 "" H 5600 4525 50  0000 C CNN
 	1    5600 4525
@@
 F 0 "RRM5" V 6080 4525 50  0000 C CNN
 F 1 "2.2k" V 6000 4525 50  0000 C CNN
-F 2 "" V 5930 4525 50  0000 C CNN
+F 2 "" V 5930 4525 50  0001 C CNN
 F 3 "" H 6000 4525 50  0000 C CNN
 	1    6000 4525
