File: Matrix.sch (KiCad schematic (older format))
At the start: 172 parts

Commit message: Rename some more keys
Saving just in case
Parts:
- removed DESC?: 1N4148WS, symbol D
- removed RESC?: 2.2k, symbol R
- added K_BACK1: MX-1U, MX_Alps_Hybrid:MX-1U, symbol MX-1U
- K_CAPS1: renamed from K_ESC?; value MX-1U -> MX-1.75U; symbol MX-1U -> MX-1.75U
- K_CAPS2: renamed from K_ESC?; value MX-1U -> MX-1.25U; symbol MX-1U -> MX-1.25U
- K_TAB1: renamed from K_ESC?; value MX-1U -> MX-1.5U; symbol MX-1U -> MX-1.5U
- gave numbers to parts that had none: 14
Changed lines of the file:
@@
 	775  1700 875  1700
 $Comp
-L MX-1U K_ESC?
+L MX-1U K_#1
 U 1 1 5983CD64
 P 1500 1525
-F 0 "K_ESC?" H 1500 1650 60  0000 C CNN
+F 0 "K_#1" H 1500 1650 60  0000 C CNN
 F 1 "MX-1U" H 1500 1575 20  0000 C CNN
 F 2 "MX_Alps_Hybrid:MX-1U" H 1475 1500 60  0001 C CNN
@@
 	1475 1700 1575 1700
 $Comp
-L MX-1U K_ESC?
+L MX-1U K_#2
 U 1 1 597DB099
 P 2200 1525
-F 0 "K_ESC?" H 2200 1650 60  0000 C CNN
+F 0 "K_#2" H 2200 1650 60  0000 C CNN
 F 1 "MX-1U" H 2200 1575 20  0000 C CNN
 F 2 "MX_Alps_Hybrid:MX-1U" H 2175 1500 60  0001 C CNN
@@
 	2175 1700 2275 1700
 $Comp
-L MX-1U K_ESC?
+L MX-1U K_#3
 U 1 1 597DB0AD
 P 2900 1525
-F 0 "K_ESC?" H 2900 1650 60  0000 C CNN
+F 0 "K_#3" H 2900 1650 60  0000 C CNN
 F 1 "MX-1U" H 2900 1575 20  0000 C CNN
 F 2 "MX_Alps_Hybrid:MX-1U" H 2875 1500 60  0001 C CNN
@@
 	2875 1700 2975 1700
 $Comp
-L MX-1U K_ESC?
+L MX-1U K_#4
 U 1 1 597DB5AD
 P 3600 1525
-F 0 "K_ESC?" H 3600 1650 60  0000 C CNN
+F 0 "K_#4" H 3600 1650 60  0000 C CNN
 F 1 "MX-1U" H 3600 1575 20  0000 C CNN
 F 2 "MX_Alps_Hybrid:MX-1U" H 3575 1500 60  0001 C CNN
@@
 	3575 1700 3675 1700
 $Comp
-L MX-1U K_ESC?
+L MX-1U K_#5
 U 1 1 597DB5C1
 P 4300 1525
-F 0 "K_ESC?" H 4300 1650 60  0000 C CNN
+F 0 "K_#5" H 4300 1650 60  0000 C CNN
 F 1 "MX-1U" H 4300 1575 20  0000 C CNN
 F 2 "MX_Alps_Hybrid:MX-1U" H 4275 1500 60  0001 C CNN
@@
 	4275 1700 4375 1700
 $Comp
-L MX-1U K_ESC?
+L MX-1U K_#6
 U 1 1 597DB5D5
 P 5000 1525
-F 0 "K_ESC?" H 5000 1650 60  0000 C CNN
+F 0 "K_#6" H 5000 1650 60  0000 C CNN
 F 1 "MX-1U" H 5000 1575 20  0000 C CNN
 F 2 "MX_Alps_Hybrid:MX-1U" H 4975 1500 60  0001 C CNN
@@
 	4975 1700 5075 1700
 $Comp
-L MX-1U K_ESC?
+L MX-1U K_#7
 U 1 1 597DB5E9
 P 5700 1525
-F 0 "K_ESC?" H 5700 1650 60  0000 C CNN
+F 0 "K_#7" H 5700 1650 60  0000 C CNN
 F 1 "MX-1U" H 5700 1575 20  0000 C CNN
 F 2 "MX_Alps_Hybrid:MX-1U" H 5675 1500 60  0001 C CNN
@@
 	5675 1700 5775 1700
 $Comp
-L MX-1U K_ESC?
+L MX-1U K_#8
 U 1 1 597DF714
 P 6400 1525
-F 0 "K_ESC?" H 6400 1650 60  0000 C CNN
+F 0 "K_#8" H 6400 1650 60  0000 C CNN
 F 1 "MX-1U" H 6400 1575 20  0000 C CNN
 F 2 "MX_Alps_Hybrid:MX-1U" H 6375 1500 60  0001 C CNN
@@
 	6375 1700 6475 1700
 $Comp
-L MX-1U K_ESC?
+L MX-1U K_#9
 U 1 1 597DF728
 P 7100 1525
-F 0 "K_ESC?" H 7100 1650 60  0000 C CNN
+F 0 "K_#9" H 7100 1650 60  0000 C CNN
 F 1 "MX-1U" H 7100 1575 20  0000 C CNN
 F 2 "MX_Alps_Hybrid:MX-1U" H 7075 1500 60  0001 C CNN
@@
 	7075 1700 7175 1700
 $Comp
-L MX-1U K_ESC?
+L MX-1U K_#0_1
 U 1 1 597DF73C
 P 7800 1525
-F 0 "K_ESC?" H 7800 1650 60  0000 C CNN
+F 0 "K_#0_1" H 7800 1650 60  0000 C CNN
 F 1 "MX-1U" H 7800 1575 20  0000 C CNN
 F 2 "MX_Alps_Hybrid:MX-1U" H 7775 1500 60  0001 C CNN
@@
 	7775 1700 7875 1700
 $Comp
-L MX-1U K_ESC?
+L MX-1U K_-1
 U 1 1 597E0014
 P 8500 1525
-F 0 "K_ESC?" H 8500 1650 60  0000 C CNN
+F 0 "K_-1" H 8500 1650 60  0000 C CNN
 F 1 "MX-1U" H 8500 1575 20  0000 C CNN
 F 2 "MX_Alps_Hybrid:MX-1U" H 8475 1500 60  0001 C CNN
@@
 	8475 1700 8575 1700
 $Comp
-L MX-1U K_ESC?
+L MX-1U K_=1
 U 1 1 597E0028
 P 9200 1525
-F 0 "K_ESC?" H 9200 1650 60  0000 C CNN
+F 0 "K_=1" H 9200 1650 60  0000 C CNN
 F 1 "MX-1U" H 9200 1575 20  0000 C CNN
 F 2 "MX_Alps_Hybrid:MX-1U" H 9175 1500 60  0001 C CNN
@@
 	9175 1700 9275 1700
 $Comp
-L MX-1U K_ESC?
+L MX-1U K_DEL1
 U 1 1 597E003C
 P 9900 1525
-F 0 "K_ESC?" H 9900 1650 60  0000 C CNN
+F 0 "K_DEL1" H 9900 1650 60  0000 C CNN
 F 1 "MX-1U" H 9900 1575 20  0000 C CNN
 F 2 "MX_Alps_Hybrid:MX-1U" H 9875 1500 60  0001 C CNN
@@
 	9875 1700 9975 1700
 $Comp
-L MX-1U K_ESC?
+L MX-1U K_SBACK1
 U 1 1 597E0050
 P 10600 1525
-F 0 "K_ESC?" H 10600 1650 60  0000 C CNN
+F 0 "K_SBACK1" H 10600 1650 60  0000 C CNN
 F 1 "MX-1U" H 10600 1575 20  0000 C CNN
 F 2 "MX_Alps_Hybrid:MX-1U" H 10575 1500 60  0001 C CNN
@@
 	10575 1700 10675 1700
 $Comp
-L MX-1U K_ESC?
+L MX-1.5U K_TAB1
 U 1 1 597E3B65
 P 1500 2075
-F 0 "K_ESC?" H 1500 2200 60  0000 C CNN
-F 1 "MX-1U" H 1500 2125 20  0000 C CNN
+F 0 "K_TAB1" H 1500 2200 60  0000 C CNN
+F 1 "MX-1.5U" H 1500 2125 20  0000 C CNN
 F 2 "MX_Alps_Hybrid:MX-1U" H 1475 2050 60  0001 C CNN
 F 3 "" H 1475 2050 60  0001 C CNN
@@
 	10575 2250 10675 2250
 $Comp
-L MX-1U K_ESC?
+L MX-1.75U K_CAPS1
 U 1 1 597E5CA5
 P 1500 2625
-F 0 "K_ESC?" H 1500 2750 60  0000 C CNN
-F 1 "MX-1U" H 1500 2675 20  0000 C CNN
+F 0 "K_CAPS1" H 1500 2750 60  0000 C CNN
+F 1 "MX-1.75U" H 1500 2675 20  0000 C CNN
 F 2 "MX_Alps_Hybrid:MX-1U" H 1475 2600 60  0001 C CNN
 F 3 "" H 1475 2600 60  0001 C CNN
@@
 	10575 2800 10675 2800
 $Comp
-L MX-1U K_ESC?
+L MX-1.25U K_CAPS2
 U 1 1 597E5DBD
 P 1500 3175
-F 0 "K_ESC?" H 1500 3300 60  0000 C CNN
-F 1 "MX-1U" H 1500 3225 20  0000 C CNN
+F 0 "K_CAPS2" H 1500 3300 60  0000 C CNN
+F 1 "MX-1.25U" H 1500 3225 20  0000 C CNN
 F 2 "MX_Alps_Hybrid:MX-1U" H 1475 3150 60  0001 C CNN
 F 3 "" H 1475 3150 60  0001 C CNN
@@
 	1    0    0    -1
 $EndComp
-$Comp
-L R RESC?
-U 1 1 597E5DC3
-P 1900 3200
-F 0 "RESC?" V 1980 3200 50  0000 C CNN
-F 1 "2.2k" V 1900 3200 50  0000 C CNN
-F 2 "" V 1830 3200 50  0001 C CNN
-F 3 "" H 1900 3200 50  0001 C CNN
-	1    1900 3200
-	0    -1   -1   0
-$EndComp
-$Comp
-L D DESC?
-U 1 1 597E5DC9
-P 1725 3350
-F 0 "DESC?" H 1725 3475 50  0000 C CNN
-F 1 "1N4148WS" H 1725 3425 20  0000 C CNN
-F 2 "" H 1725 3350 50  0001 C CNN
-F 3 "" H 1725 3350 50  0001 C CNN
-	1    1725 3350
-	-1   0    0    1
-$EndComp
-Wire Wire Line
-	1750 3200 1625 3200
-Wire Wire Line
-	1475 3350 1575 3350
 $Comp
 L MX-1U K_ESC?
@@
 	1    0    0    -1
 $EndComp
+$Comp
+L MX-1U K_BACK1
+U 1 1 59800CF4
+P 9900 975
+F 0 "K_BACK1" H 9900 1100 60  0000 C CNN
+F 1 "MX-1U" H 9900 1025 20  0000 C CNN
+F 2 "MX_Alps_Hybrid:MX-1U" H 9875 950 60  0001 C CNN
+F 3 "" H 9875 950 60  0001 C CNN
+	1    9900 975
+	1    0    0    -1
+$EndComp

Commit message: Rename 2nd row keys
Parts:
- gave numbers to parts that had none: 13
Changed lines of the file:
@@
 	1475 2250 1575 2250
 $Comp
-L MX-1U K_ESC?
+L MX-1U K_Q1
 U 1 1 597E3B79
 P 2200 2075
-F 0 "K_ESC?" H 2200 2200 60  0000 C CNN
+F 0 "K_Q1" H 2200 2200 60  0000 C CNN
 F 1 "MX-1U" H 2200 2125 20  0000 C CNN
 F 2 "MX_Alps_Hybrid:MX-1U" H 2175 2050 60  0001 C CNN
@@
 	2175 2250 2275 2250
 $Comp
-L MX-1U K_ESC?
+L MX-1U K_W1
 U 1 1 597E3B8D
 P 2900 2075
-F 0 "K_ESC?" H 2900 2200 60  0000 C CNN
+F 0 "K_W1" H 2900 2200 60  0000 C CNN
 F 1 "MX-1U" H 2900 2125 20  0000 C CNN
 F 2 "MX_Alps_Hybrid:MX-1U" H 2875 2050 60  0001 C CNN
@@
 	2875 2250 2975 2250
 $Comp
-L MX-1U K_ESC?
+L MX-1U K_E1
 U 1 1 597E3BA1
 P 3600 2075
-F 0 "K_ESC?" H 3600 2200 60  0000 C CNN
+F 0 "K_E1" H 3600 2200 60  0000 C CNN
 F 1 "MX-1U" H 3600 2125 20  0000 C CNN
 F 2 "MX_Alps_Hybrid:MX-1U" H 3575 2050 60  0001 C CNN
@@
 	3575 2250 3675 2250
 $Comp
-L MX-1U K_ESC?
+L MX-1U K_R1
 U 1 1 597E3BB5
 P 4300 2075
-F 0 "K_ESC?" H 4300 2200 60  0000 C CNN
+F 0 "K_R1" H 4300 2200 60  0000 C CNN
 F 1 "MX-1U" H 4300 2125 20  0000 C CNN
 F 2 "MX_Alps_Hybrid:MX-1U" H 4275 2050 60  0001 C CNN
@@
 	4275 2250 4375 2250
 $Comp
-L MX-1U K_ESC?
+L MX-1U K_T1
 U 1 1 597E3BC9
 P 5000 2075
-F 0 "K_ESC?" H 5000 2200 60  0000 C CNN
+F 0 "K_T1" H 5000 2200 60  0000 C CNN
 F 1 "MX-1U" H 5000 2125 20  0000 C CNN
 F 2 "MX_Alps_Hybrid:MX-1U" H 4975 2050 60  0001 C CNN
@@
 	4975 2250 5075 2250
 $Comp
-L MX-1U K_ESC?
+L MX-1U K_Y1
 U 1 1 597E3BDD
 P 5700 2075
-F 0 "K_ESC?" H 5700 2200 60  0000 C CNN
+F 0 "K_Y1" H 5700 2200 60  0000 C CNN
 F 1 "MX-1U" H 5700 2125 20  0000 C CNN
 F 2 "MX_Alps_Hybrid:MX-1U" H 5675 2050 60  0001 C CNN
@@
 	5675 2250 5775 2250
 $Comp
-L MX-1U K_ESC?
+L MX-1U K_U1
 U 1 1 597E3BF1
 P 6400 2075
-F 0 "K_ESC?" H 6400 2200 60  0000 C CNN
+F 0 "K_U1" H 6400 2200 60  0000 C CNN
 F 1 "MX-1U" H 6400 2125 20  0000 C CNN
 F 2 "MX_Alps_Hybrid:MX-1U" H 6375 2050 60  0001 C CNN
@@
 	6375 2250 6475 2250
 $Comp
-L MX-1U K_ESC?
+L MX-1U K_I1
 U 1 1 597E3C05
 P 7100 2075
-F 0 "K_ESC?" H 7100 2200 60  0000 C CNN
+F 0 "K_I1" H 7100 2200 60  0000 C CNN
 F 1 "MX-1U" H 7100 2125 20  0000 C CNN
 F 2 "MX_Alps_Hybrid:MX-1U" H 7075 2050 60  0001 C CNN
@@
 	7075 2250 7175 2250
 $Comp
-L MX-1U K_ESC?
+L MX-1U K_O1
 U 1 1 597E3C19
 P 7800 2075
-F 0 "K_ESC?" H 7800 2200 60  0000 C CNN
+F 0 "K_O1" H 7800 2200 60  0000 C CNN
 F 1 "MX-1U" H 7800 2125 20  0000 C CNN
 F 2 "MX_Alps_Hybrid:MX-1U" H 7775 2050 60  0001 C CNN
@@
 	7775 2250 7875 2250
 $Comp
-L MX-1U K_ESC?
+L MX-1U K_P1
 U 1 1 597E3C2D
 P 8500 2075
-F 0 "K_ESC?" H 8500 2200 60  0000 C CNN
+F 0 "K_P1" H 8500 2200 60  0000 C CNN
 F 1 "MX-1U" H 8500 2125 20  0000 C CNN
 F 2 "MX_Alps_Hybrid:MX-1U" H 8475 2050 60  0001 C CNN
@@
 	8475 2250 8575 2250
 $Comp
-L MX-1U K_ESC?
+L MX-1U K_[1
 U 1 1 597E3C41
 P 9200 2075
-F 0 "K_ESC?" H 9200 2200 60  0000 C CNN
+F 0 "K_[1" H 9200 2200 60  0000 C CNN
 F 1 "MX-1U" H 9200 2125 20  0000 C CNN
 F 2 "MX_Alps_Hybrid:MX-1U" H 9175 2050 60  0001 C CNN
@@
 	9175 2250 9275 2250
 $Comp
-L MX-1U K_ESC?
+L MX-1U K_]1
 U 1 1 597E3C55
 P 9900 2075
-F 0 "K_ESC?" H 9900 2200 60  0000 C CNN
+F 0 "K_]1" H 9900 2200 60  0000 C CNN
 F 1 "MX-1U" H 9900 2125 20  0000 C CNN
 F 2 "MX_Alps_Hybrid:MX-1U" H 9875 2050 60  0001 C CNN
@@
 	9875 2250 9975 2250
 $Comp
-L MX-1U K_ESC?
+L MX-1U K_\1
 U 1 1 597E3C69
 P 10600 2075
-F 0 "K_ESC?" H 10600 2200 60  0000 C CNN
+F 0 "K_\\1" H 10600 2200 60  0000 C CNN
 F 1 "MX-1U" H 10600 2125 20  0000 C CNN
 F 2 "MX_Alps_Hybrid:MX-1U" H 10575 2050 60  0001 C CNN

Commit message: Rename 3rd row
Parts:
- gave numbers to parts that had none: 13
Changed lines of the file:
@@
 	1475 2800 1575 2800
 $Comp
-L MX-1U K_ESC?
+L MX-1U K_A1
 U 1 1 597E5CB9
 P 2200 2625
-F 0 "K_ESC?" H 2200 2750 60  0000 C CNN
+F 0 "K_A1" H 2200 2750 60  0000 C CNN
 F 1 "MX-1U" H 2200 2675 20  0000 C CNN
 F 2 "MX_Alps_Hybrid:MX-1U" H 2175 2600 60  0001 C CNN
@@
 	2175 2800 2275 2800
 $Comp
-L MX-1U K_ESC?
+L MX-1U K_S1
 U 1 1 597E5CCD
 P 2900 2625
-F 0 "K_ESC?" H 2900 2750 60  0000 C CNN
+F 0 "K_S1" H 2900 2750 60  0000 C CNN
 F 1 "MX-1U" H 2900 2675 20  0000 C CNN
 F 2 "MX_Alps_Hybrid:MX-1U" H 2875 2600 60  0001 C CNN
@@
 	2875 2800 2975 2800
 $Comp
-L MX-1U K_ESC?
+L MX-1U K_D1
 U 1 1 597E5CE1
 P 3600 2625
-F 0 "K_ESC?" H 3600 2750 60  0000 C CNN
+F 0 "K_D1" H 3600 2750 60  0000 C CNN
 F 1 "MX-1U" H 3600 2675 20  0000 C CNN
 F 2 "MX_Alps_Hybrid:MX-1U" H 3575 2600 60  0001 C CNN
@@
 	3575 2800 3675 2800
 $Comp
-L MX-1U K_ESC?
+L MX-1U K_F1
 U 1 1 597E5CF5
 P 4300 2625
-F 0 "K_ESC?" H 4300 2750 60  0000 C CNN
+F 0 "K_F1" H 4300 2750 60  0000 C CNN
 F 1 "MX-1U" H 4300 2675 20  0000 C CNN
 F 2 "MX_Alps_Hybrid:MX-1U" H 4275 2600 60  0001 C CNN
@@
 	4275 2800 4375 2800
 $Comp
-L MX-1U K_ESC?
+L MX-1U K_G1
 U 1 1 597E5D09
 P 5000 2625
-F 0 "K_ESC?" H 5000 2750 60  0000 C CNN
+F 0 "K_G1" H 5000 2750 60  0000 C CNN
 F 1 "MX-1U" H 5000 2675 20  0000 C CNN
 F 2 "MX_Alps_Hybrid:MX-1U" H 4975 2600 60  0001 C CNN
@@
 	4975 2800 5075 2800
 $Comp
-L MX-1U K_ESC?
+L MX-1U K_H1
 U 1 1 597E5D1D
 P 5700 2625
-F 0 "K_ESC?" H 5700 2750 60  0000 C CNN
+F 0 "K_H1" H 5700 2750 60  0000 C CNN
 F 1 "MX-1U" H 5700 2675 20  0000 C CNN
 F 2 "MX_Alps_Hybrid:MX-1U" H 5675 2600 60  0001 C CNN
@@
 	5675 2800 5775 2800
 $Comp
-L MX-1U K_ESC?
+L MX-1U K_J1
 U 1 1 597E5D31
 P 6400 2625
-F 0 "K_ESC?" H 6400 2750 60  0000 C CNN
+F 0 "K_J1" H 6400 2750 60  0000 C CNN
 F 1 "MX-1U" H 6400 2675 20  0000 C CNN
 F 2 "MX_Alps_Hybrid:MX-1U" H 6375 2600 60  0001 C CNN
@@
 	6375 2800 6475 2800
 $Comp
-L MX-1U K_ESC?
+L MX-1U K_K1
 U 1 1 597E5D45
 P 7100 2625
-F 0 "K_ESC?" H 7100 2750 60  0000 C CNN
+F 0 "K_K1" H 7100 2750 60  0000 C CNN
 F 1 "MX-1U" H 7100 2675 20  0000 C CNN
 F 2 "MX_Alps_Hybrid:MX-1U" H 7075 2600 60  0001 C CNN
@@
 	7075 2800 7175 2800
 $Comp
-L MX-1U K_ESC?
+L MX-1U K_L1
 U 1 1 597E5D59
 P 7800 2625
-F 0 "K_ESC?" H 7800 2750 60  0000 C CNN
+F 0 "K_L1" H 7800 2750 60  0000 C CNN
 F 1 "MX-1U" H 7800 2675 20  0000 C CNN
 F 2 "MX_Alps_Hybrid:MX-1U" H 7775 2600 60  0001 C CNN
@@
 	7775 2800 7875 2800
 $Comp
-L MX-1U K_ESC?
+L MX-1U K_;1
 U 1 1 597E5D6D
 P 8500 2625
-F 0 "K_ESC?" H 8500 2750 60  0000 C CNN
+F 0 "K_;1" H 8500 2750 60  0000 C CNN
 F 1 "MX-1U" H 8500 2675 20  0000 C CNN
 F 2 "MX_Alps_Hybrid:MX-1U" H 8475 2600 60  0001 C CNN
@@
 	8475 2800 8575 2800
 $Comp
-L MX-1U K_ESC?
+L MX-1U K_'1
 U 1 1 597E5D81
 P 9200 2625
-F 0 "K_ESC?" H 9200 2750 60  0000 C CNN
+F 0 "K_'1" H 9200 2750 60  0000 C CNN
 F 1 "MX-1U" H 9200 2675 20  0000 C CNN
 F 2 "MX_Alps_Hybrid:MX-1U" H 9175 2600 60  0001 C CNN
@@
 	9175 2800 9275 2800
 $Comp
-L MX-1U K_ESC?
+L MX-1U K_ISO`1
 U 1 1 597E5D95
 P 9900 2625
-F 0 "K_ESC?" H 9900 2750 60  0000 C CNN
+F 0 "K_ISO`1" H 9900 2750 60  0000 C CNN
 F 1 "MX-1U" H 9900 2675 20  0000 C CNN
 F 2 "MX_Alps_Hybrid:MX-1U" H 9875 2600 60  0001 C CNN
@@
 	9875 2800 9975 2800
 $Comp
-L MX-1U K_ESC?
+L MX-1U K_ENTER1
 U 1 1 597E5DA9
 P 10600 2625
-F 0 "K_ESC?" H 10600 2750 60  0000 C CNN
+F 0 "K_ENTER1" H 10600 2750 60  0000 C CNN
 F 1 "MX-1U" H 10600 2675 20  0000 C CNN
 F 2 "MX_Alps_Hybrid:MX-1U" H 10575 2600 60  0001 C CNN

Commit message: Finish renaming keys
Now onto resistors
Parts:
- gave numbers to parts that had none: 20
Changed lines of the file:
@@
 $EndComp
 $Comp
-L MX-1U K_ESC?
+L MX-1U K_Z1
 U 1 1 597E5DD1
 P 2200 3175
-F 0 "K_ESC?" H 2200 3300 60  0000 C CNN
+F 0 "K_Z1" H 2200 3300 60  0000 C CNN
 F 1 "MX-1U" H 2200 3225 20  0000 C CNN
 F 2 "MX_Alps_Hybrid:MX-1U" H 2175 3150 60  0001 C CNN
@@
 	2175 3350 2275 3350
 $Comp
-L MX-1U K_ESC?
+L MX-1U K_X1
 U 1 1 597E5DE5
 P 2900 3175
-F 0 "K_ESC?" H 2900 3300 60  0000 C CNN
+F 0 "K_X1" H 2900 3300 60  0000 C CNN
 F 1 "MX-1U" H 2900 3225 20  0000 C CNN
 F 2 "MX_Alps_Hybrid:MX-1U" H 2875 3150 60  0001 C CNN
@@
 	2875 3350 2975 3350
 $Comp
-L MX-1U K_ESC?
+L MX-1U K_C1
 U 1 1 597E5DF9
 P 3600 3175
-F 0 "K_ESC?" H 3600 3300 60  0000 C CNN
+F 0 "K_C1" H 3600 3300 60  0000 C CNN
 F 1 "MX-1U" H 3600 3225 20  0000 C CNN
 F 2 "MX_Alps_Hybrid:MX-1U" H 3575 3150 60  0001 C CNN
@@
 	3575 3350 3675 3350
 $Comp
-L MX-1U K_ESC?
+L MX-1U K_V1
 U 1 1 597E5E0D
 P 4300 3175
-F 0 "K_ESC?" H 4300 3300 60  0000 C CNN
+F 0 "K_V1" H 4300 3300 60  0000 C CNN
 F 1 "MX-1U" H 4300 3225 20  0000 C CNN
 F 2 "MX_Alps_Hybrid:MX-1U" H 4275 3150 60  0001 C CNN
@@
 	4275 3350 4375 3350
 $Comp
-L MX-1U K_ESC?
+L MX-1U K_B1
 U 1 1 597E5E21
 P 5000 3175
-F 0 "K_ESC?" H 5000 3300 60  0000 C CNN
+F 0 "K_B1" H 5000 3300 60  0000 C CNN
 F 1 "MX-1U" H 5000 3225 20  0000 C CNN
 F 2 "MX_Alps_Hybrid:MX-1U" H 4975 3150 60  0001 C CNN
@@
 	4975 3350 5075 3350
 $Comp
-L MX-1U K_ESC?
+L MX-1U K_N1
 U 1 1 597E5E35
 P 5700 3175
-F 0 "K_ESC?" H 5700 3300 60  0000 C CNN
+F 0 "K_N1" H 5700 3300 60  0000 C CNN
 F 1 "MX-1U" H 5700 3225 20  0000 C CNN
 F 2 "MX_Alps_Hybrid:MX-1U" H 5675 3150 60  0001 C CNN
@@
 	5675 3350 5775 3350
 $Comp
-L MX-1U K_ESC?
+L MX-1U K_M1
 U 1 1 597E5E49
 P 6400 3175
-F 0 "K_ESC?" H 6400 3300 60  0000 C CNN
+F 0 "K_M1" H 6400 3300 60  0000 C CNN
 F 1 "MX-1U" H 6400 3225 20  0000 C CNN
 F 2 "MX_Alps_Hybrid:MX-1U" H 6375 3150 60  0001 C CNN
@@
 	6375 3350 6475 3350
 $Comp
-L MX-1U K_ESC?
+L MX-1U K_,1
 U 1 1 597E5E5D
 P 7100 3175
-F 0 "K_ESC?" H 7100 3300 60  0000 C CNN
+F 0 "K_,1" H 7100 3300 60  0000 C CNN
 F 1 "MX-1U" H 7100 3225 20  0000 C CNN
 F 2 "MX_Alps_Hybrid:MX-1U" H 7075 3150 60  0001 C CNN
@@
 	7075 3350 7175 3350
 $Comp
-L MX-1U K_ESC?
+L MX-1U K_.1
 U 1 1 597E5E71
 P 7800 3175
-F 0 "K_ESC?" H 7800 3300 60  0000 C CNN
+F 0 "K_.1" H 7800 3300 60  0000 C CNN
 F 1 "MX-1U" H 7800 3225 20  0000 C CNN
 F 2 "MX_Alps_Hybrid:MX-1U" H 7775 3150 60  0001 C CNN
@@
 	7775 3350 7875 3350
 $Comp
-L MX-1U K_ESC?
+L MX-1U K_?1
 U 1 1 597E5E85
 P 8500 3175
-F 0 "K_ESC?" H 8500 3300 60  0000 C CNN
+F 0 "K_?1" H 8500 3300 60  0000 C CNN
 F 1 "MX-1U" H 8500 3225 20  0000 C CNN
 F 2 "MX_Alps_Hybrid:MX-1U" H 8475 3150 60  0001 C CNN
@@
 	8475 3350 8575 3350
 $Comp
-L MX-1U K_ESC?
+L MX-1U K_Z2
 U 1 1 597EB000
 P 2200 3725
-F 0 "K_ESC?" H 2200 3850 60  0000 C CNN
+F 0 "K_Z2" H 2200 3850 60  0000 C CNN
 F 1 "MX-1U" H 2200 3775 20  0000 C CNN
 F 2 "MX_Alps_Hybrid:MX-1U" H 2175 3700 60  0001 C CNN
@@
 $EndComp
 $Comp
-L MX-1U K_ESC?
+L MX-1U K_X2
 U 1 1 597EB014
 P 2900 3725
-F 0 "K_ESC?" H 2900 3850 60  0000 C CNN
+F 0 "K_X2" H 2900 3850 60  0000 C CNN
 F 1 "MX-1U" H 2900 3775 20  0000 C CNN
 F 2 "MX_Alps_Hybrid:MX-1U" H 2875 3700 60  0001 C CNN
@@
 $EndComp
 $Comp
-L MX-1U K_ESC?
+L MX-1U K_C2
 U 1 1 597EB028
 P 3600 3725
-F 0 "K_ESC?" H 3600 3850 60  0000 C CNN
+F 0 "K_C2" H 3600 3850 60  0000 C CNN
 F 1 "MX-1U" H 3600 3775 20  0000 C CNN
 F 2 "MX_Alps_Hybrid:MX-1U" H 3575 3700 60  0001 C CNN
@@
 $EndComp
 $Comp
-L MX-1U K_ESC?
+L MX-1U K_V2
 U 1 1 597EB03C
 P 4300 3725
-F 0 "K_ESC?" H 4300 3850 60  0000 C CNN
+F 0 "K_V2" H 4300 3850 60  0000 C CNN
 F 1 "MX-1U" H 4300 3775 20  0000 C CNN
 F 2 "MX_Alps_Hybrid:MX-1U" H 4275 3700 60  0001 C CNN
@@
 $EndComp
 $Comp
-L MX-1U K_ESC?
+L MX-1U K_B2
 U 1 1 597EB050
 P 5000 3725
-F 0 "K_ESC?" H 5000 3850 60  0000 C CNN
+F 0 "K_B2" H 5000 3850 60  0000 C CNN
 F 1 "MX-1U" H 5000 3775 20  0000 C CNN
 F 2 "MX_Alps_Hybrid:MX-1U" H 4975 3700 60  0001 C CNN
@@
 $EndComp
 $Comp
-L MX-1U K_ESC?
+L MX-1U K_N2
 U 1 1 597EB064
 P 5700 3725
-F 0 "K_ESC?" H 5700 3850 60  0000 C CNN
+F 0 "K_N2" H 5700 3850 60  0000 C CNN
 F 1 "MX-1U" H 5700 3775 20  0000 C CNN
 F 2 "MX_Alps_Hybrid:MX-1U" H 5675 3700 60  0001 C CNN
@@
 $EndComp
 $Comp
-L MX-1U K_ESC?
+L MX-1U K_M2
 U 1 1 597EB078
 P 6400 3725
-F 0 "K_ESC?" H 6400 3850 60  0000 C CNN
+F 0 "K_M2" H 6400 3850 60  0000 C CNN
 F 1 "MX-1U" H 6400 3775 20  0000 C CNN
 F 2 "MX_Alps_Hybrid:MX-1U" H 6375 3700 60  0001 C CNN
@@
 $EndComp
 $Comp
-L MX-1U K_ESC?
+L MX-1U K_,2
 U 1 1 597EB08C
 P 7100 3725
-F 0 "K_ESC?" H 7100 3850 60  0000 C CNN
+F 0 "K_,2" H 7100 3850 60  0000 C CNN
 F 1 "MX-1U" H 7100 3775 20  0000 C CNN
 F 2 "MX_Alps_Hybrid:MX-1U" H 7075 3700 60  0001 C CNN
@@
 $EndComp
 $Comp
-L MX-1U K_ESC?
+L MX-1U K_.2
 U 1 1 597EB0A0
 P 7800 3725
-F 0 "K_ESC?" H 7800 3850 60  0000 C CNN
+F 0 "K_.2" H 7800 3850 60  0000 C CNN
 F 1 "MX-1U" H 7800 3775 20  0000 C CNN
 F 2 "MX_Alps_Hybrid:MX-1U" H 7775 3700 60  0001 C CNN
@@
 $EndComp
 $Comp
-L MX-1U K_ESC?
+L MX-1U K_?2
 U 1 1 597EB0B4
 P 8500 3725
-F 0 "K_ESC?" H 8500 3850 60  0000 C CNN
+F 0 "K_?2" H 8500 3850 60  0000 C CNN
 F 1 "MX-1U" H 8500 3775 20  0000 C CNN
 F 2 "MX_Alps_Hybrid:MX-1U" H 8475 3700 60  0001 C CNN
