File: Kairos.kicad_pcb (KiCad board)
At the start: 2 copper layers, 285 x 94.6 mm, 142 parts, among them Q1 NSS40301MZ4T1G, SW1 SW_RST1, U1 ATMEGA32U2-AU, Y1 Crystal_GND24

Commit message: Flip again since KiCad ignored changes
Parts:
- K_BACK1: footprint MX_Alps_Hybrid:MX-2U -> MX_Alps_Hybrid:MX-1U
- K_CAPS1: footprint MX_Alps_Hybrid:MX-1.75U -> MX_Alps_Hybrid:MX-1U
- K_CAPS2, K_SENTER1: footprint MX_Alps_Hybrid:MX-1.25U -> MX_Alps_Hybrid:MX-1U
- K_ENTER1: footprint MX_Alps_Hybrid:MX-2.25U -> MX_Alps_Hybrid:MX-1U
- K_ISOENTER1: footprint MX_Alps_Hybrid:MX-ISO-Combined -> MX_Alps_Hybrid:MX-1U
- K_SP1, K_SP3: footprint MX_Alps_Hybrid:MX-7U -> MX_Alps_Hybrid:MX-7U-ReversedStabilizers
- K_SP2: footprint MX_Alps_Hybrid:MX-6.25U -> MX_Alps_Hybrid:MX-6.25U-ReversedStabilizers
- K_TAB1, K_\1: footprint MX_Alps_Hybrid:MX-1.5U -> MX_Alps_Hybrid:MX-1U
- turned K_SP1 to 0 degrees
- turned K_SP2 to 0 degrees
- turned K_SP3 to 0 degrees

Commit message: Stack bottom row, move HHKB layout out of the way temporarily
Parts:
- added K_SP3_Extra1: MX-6U, MX_Alps_Hybrid:MX-6U-7UOverlay, F.Cu at (141.3, 326.2)
- moved K_LM1 173.9 mm to (19.8, 326.2)
- moved K_LM3 173.9 mm to (43.7, 326.2)
- moved K_LM6 173.9 mm to (67.5, 326.2)
- moved K_RM10 173.9 mm to (281.8, 326.2)
- moved K_RM2 173.9 mm to (210.3, 326.2)
- moved K_RM4 173.9 mm to (234.2, 326.2)
- moved K_RM6 173.9 mm to (258.0, 326.2)
- moved K_SP2 173.9 mm to (138.9, 326.2)
- moved K_RM1 154.8 mm to (208.0, 326.2)
- moved K_RM11 154.8 mm to (284.2, 326.2)
- moved K_RM3 154.8 mm to (227.0, 326.2)
- moved K_RM8 154.8 mm to (246.1, 326.2)
- moved K_RM9 154.8 mm to (265.1, 326.2)
- moved K_LM2 116.7 mm to (22.2, 326.2)
- moved K_LM4 116.7 mm to (46.0, 326.2)
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Changed lines of the file:
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@@
     (tracks 278)
     (zones 0)
-    (modules 142)
+    (modules 143)
     (nets 190)
   )
@@
   )
   (module MX_Alps_Hybrid:MX-6U locked (layer F.Cu)
-    (at 139.065 107.15625)
+    (at 139.065 150.01875)
     (fp_text reference K_SP15 (at 9.525 3.175) (layer F.SilkS)
       (effects (font (size 1 1) (thickness 0.15)))
@@
   )
   (module MX_Alps_Hybrid:MX-1.5U locked (layer F.Cu)
-    (at 210.5025 107.15625)
+    (at 210.5025 150.01875)
     (fp_text reference K_RM15 (at 0 3.175) (layer F.SilkS)
       (effects (font (size 1 1) (thickness 0.15)))
@@
   )
   (module MX_Alps_Hybrid:MX-1.5U locked (layer F.Cu)
-    (at 67.6275 107.15625)
+    (at 67.6275 150.01875)
     (fp_text reference K_LM9 (at 0 3.175) (layer F.SilkS)
       (effects (font (size 1 1) (thickness 0.15)))
@@
   )
   (module MX_Alps_Hybrid:MX-1.5U (layer F.Cu)
-    (at 66.675 209.55)
+    (at 69.85 326.23125)
     (fp_text reference K_LM7 (at 0 3.175) (layer F.SilkS)
       (effects (font (size 1 1) (thickness 0.15)))
@@
   )
   (module MX_Alps_Hybrid:MX-1.5U (layer F.Cu)
-    (at 47.625 304.8)
+    (at 50.8 326.23125)
     (fp_text reference K_LM5 (at 0 3.175) (layer F.SilkS)
       (effects (font (size 1 1) (thickness 0.15)))
@@
   )
   (module MX_Alps_Hybrid:MX-1.5U (layer F.Cu)
-    (at 19.05 209.55)
+    (at 22.225 326.23125)
     (fp_text reference K_LM2 (at 0 3.175) (layer F.SilkS)
       (effects (font (size 1 1) (thickness 0.15)))
@@
   )
   (module MX_Alps_Hybrid:MX-1.5U (layer F.Cu)
-    (at 276.225 266.7)
+    (at 279.4 326.23125)
     (fp_text reference K_RM12 (at 0 3.175) (layer F.SilkS)
       (effects (font (size 1 1) (thickness 0.15)))
@@
   )
   (module MX_Alps_Hybrid:MX-1.5U (layer F.Cu)
-    (at 228.6 266.7)
+    (at 231.775 326.23125)
     (fp_text reference K_RM5 (at 0 3.175) (layer F.SilkS)
       (effects (font (size 1 1) (thickness 0.15)))
@@
   )
   (module MX_Alps_Hybrid:MX-1.25U (layer F.Cu)
-    (at 64.29375 152.4)
+    (at 67.46875 326.23125)
     (fp_text reference K_LM6 (at 0 3.175) (layer F.SilkS)
       (effects (font (size 1 1) (thickness 0.15)))
@@
   )
   (module MX_Alps_Hybrid:MX-1.25U (layer F.Cu)
-    (at 40.48125 152.4)
+    (at 43.65625 326.23125)
     (fp_text reference K_LM3 (at 0 3.175) (layer F.SilkS)
       (effects (font (size 1 1) (thickness 0.15)))
@@
   )
   (module MX_Alps_Hybrid:MX-1.25U (layer F.Cu)
-    (at 16.66875 152.4)
+    (at 19.84375 326.23125)
     (fp_text reference K_LM1 (at 0 3.175) (layer F.SilkS)
       (effects (font (size 1 1) (thickness 0.15)))
@@
   )
   (module MX_Alps_Hybrid:MX-1.25U (layer F.Cu)
-    (at 278.60625 152.4)
+    (at 281.78125 326.23125)
     (fp_text reference K_RM10 (at 0 3.175) (layer F.SilkS)
       (effects (font (size 1 1) (thickness 0.15)))
@@
   )
   (module MX_Alps_Hybrid:MX-1.25U (layer F.Cu)
-    (at 254.79375 152.4)
+    (at 257.96875 326.23125)
     (fp_text reference K_RM6 (at 0 3.175) (layer F.SilkS)
       (effects (font (size 1 1) (thickness 0.15)))
@@
   )
   (module MX_Alps_Hybrid:MX-1.25U (layer F.Cu)
-    (at 230.98125 152.4)
+    (at 234.15625 326.23125)
     (fp_text reference K_RM4 (at 0 3.175) (layer F.SilkS)
       (effects (font (size 1 1) (thickness 0.15)))
@@
   )
   (module MX_Alps_Hybrid:MX-1.25U (layer F.Cu)
-    (at 207.16875 152.4)
+    (at 210.34375 326.23125)
     (fp_text reference K_RM2 (at 0 3.175) (layer F.SilkS)
       (effects (font (size 1 1) (thickness 0.15)))
@@
   )
   (module MX_Alps_Hybrid:MX-1U (layer F.Cu)
-    (at 204.7875 171.45)
+    (at 207.9625 326.23125)
     (fp_text reference K_RM1 (at 0 3.175) (layer F.SilkS)
       (effects (font (size 1 1) (thickness 0.15)))
@@
   )
   (module MX_Alps_Hybrid:MX-1U (layer F.Cu)
-    (at 223.8375 171.45)
+    (at 227.0125 326.23125)
     (fp_text reference K_RM3 (at 0 3.175) (layer F.SilkS)
       (effects (font (size 1 1) (thickness 0.15)))
@@
   )
   (module MX_Alps_Hybrid:MX-1U (layer F.Cu)
-    (at 252.4125 266.7)
+    (at 255.5875 326.23125)
     (fp_text reference K_RM7 (at 0 3.175) (layer F.SilkS)
       (effects (font (size 1 1) (thickness 0.15)))
@@
   )
   (module MX_Alps_Hybrid:MX-1U (layer F.Cu)
-    (at 242.8875 171.45)
+    (at 246.0625 326.23125)
     (fp_text reference K_RM8 (at 0 3.175) (layer F.SilkS)
       (effects (font (size 1 1) (thickness 0.15)))
@@
   )
   (module MX_Alps_Hybrid:MX-1U (layer F.Cu)
-    (at 261.9375 171.45)
+    (at 265.1125 326.23125)
     (fp_text reference K_RM9 (at 0 3.175) (layer F.SilkS)
       (effects (font (size 1 1) (thickness 0.15)))
@@
   )
   (module MX_Alps_Hybrid:MX-1U (layer F.Cu)
-    (at 280.9875 171.45)
+    (at 284.1625 326.23125)
     (fp_text reference K_RM11 (at 0 3.175) (layer F.SilkS)
       (effects (font (size 1 1) (thickness 0.15)))
@@
   )
   (module MX_Alps_Hybrid:MX-1U (layer F.Cu)
-    (at 42.8625 209.55)
+    (at 46.0375 326.23125)
     (fp_text reference K_LM4 (at 0 3.175) (layer F.SilkS)
       (effects (font (size 1 1) (thickness 0.15)))
@@
   )
   (module MX_Alps_Hybrid:MX-1U locked (layer F.Cu)
-    (at 43.815 107.15625)
+    (at 43.815 150.01875)
     (fp_text reference K_LM8 (at 0 3.175) (layer F.SilkS)
       (effects (font (size 1 1) (thickness 0.15)))
@@
   )
   (module MX_Alps_Hybrid:MX-1U locked (layer F.Cu)
-    (at 234.315 107.15625)
+    (at 234.315 150.01875)
     (fp_text reference K_RM16 (at 0 3.175) (layer F.SilkS)
       (effects (font (size 1 1) (thickness 0.15)))
@@
   )
   (module MX_Alps_Hybrid:MX-7U-ReversedStabilizers (layer F.Cu)
-    (at 128.5875 304.8)
+    (at 131.7625 326.23125)
     (fp_text reference K_SP1 (at 0 3.175) (layer F.SilkS)
       (effects (font (size 1 1) (thickness 0.15)))
@@
   )
   (module MX_Alps_Hybrid:MX-6.25U-ReversedStabilizers (layer F.Cu)
-    (at 135.73125 152.4)
+    (at 138.90625 326.23125)
     (fp_text reference K_SP2 (at 0 3.175) (layer F.SilkS)
       (effects (font (size 1 1) (thickness 0.15)))
@@
   )
   (module MX_Alps_Hybrid:MX-7U-ReversedStabilizers (layer F.Cu)
-    (at 147.6375 209.55)
+    (at 150.8125 326.23125)
     (fp_text reference K_SP3 (at 0 3.175) (layer F.SilkS)
       (effects (font (size 1 1) (thickness 0.15)))
@@
     (pad "" np_thru_hole circle (at 5.08 0 48.0996) (size 1.7018 1.7018) (drill 1.7018) (layers *.Cu *.Mask))
   )
+  (module MX_Alps_Hybrid:MX-6U-7UOverlay (layer F.Cu)
+    (at 141.2875 326.23125)
+    (fp_text reference K_SP3_Extra1 (at 9.525 3.175) (layer F.SilkS)
+      (effects (font (size 1 1) (thickness 0.15)))
+    )
+    (fp_text value MX-6U (at 9.525 -7.9375) (layer Dwgs.User)
+      (effects (font (size 1 1) (thickness 0.15)))
+    )
+    (fp_line (start -57.15 -9.525) (end 57.15 -9.525) (layer Dwgs.User) (width 0.15))
+    (fp_line (start 57.15 -9.525) (end 57.15 9.525) (layer Dwgs.User) (width 0.15))
+    (fp_line (start -57.15 9.525) (end 57.15 9.525) (layer Dwgs.User) (width 0.15))
+    (fp_line (start -57.15 9.525) (end -57.15 -9.525) (layer Dwgs.User) (width 0.15))
+    (pad "" np_thru_hole circle (at 47.625 6.985) (size 3.048 3.048) (drill 3.048) (layers *.Cu *.Mask))
+    (pad "" np_thru_hole circle (at 47.625 -8.255) (size 3.9878 3.9878) (drill 3.9878) (layers *.Cu *.Mask))
+  )
   (gr_text "RS7 already\ncovered" (at 416.71875 88.10625) (layer Dwgs.User)

Commit message: Move stock XD60 layout (+SP3 7U) to main layout
Parts:
- moved K_LM1 219.1 mm to (16.7, 107.2)
- moved K_LM2 219.1 mm to (19.1, 107.2)
- moved K_LM3 219.1 mm to (40.5, 107.2)
- moved K_LM4 219.1 mm to (42.9, 107.2)
- moved K_LM5 219.1 mm to (47.6, 107.2)
- moved K_LM6 219.1 mm to (64.3, 107.2)
- moved K_LM7 219.1 mm to (66.7, 107.2)
- moved K_RM1 219.1 mm to (204.8, 107.2)
- moved K_RM10 219.1 mm to (278.6, 107.2)
- moved K_RM11 219.1 mm to (281.0, 107.2)
- moved K_RM12 219.1 mm to (276.2, 107.2)
- moved K_RM2 219.1 mm to (207.2, 107.2)
- moved K_RM3 219.1 mm to (223.8, 107.2)
- moved K_RM4 219.1 mm to (231.0, 107.2)
- moved K_RM5 219.1 mm to (228.6, 107.2)
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Changed lines of the file:
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@@
   )
   (module MX_Alps_Hybrid:MX-1.5U (layer F.Cu)
-    (at 69.85 326.23125)
+    (at 66.675 107.15625)
     (fp_text reference K_LM7 (at 0 3.175) (layer F.SilkS)
       (effects (font (size 1 1) (thickness 0.15)))
@@
   )
   (module MX_Alps_Hybrid:MX-1.5U (layer F.Cu)
-    (at 50.8 326.23125)
+    (at 47.625 107.15625)
     (fp_text reference K_LM5 (at 0 3.175) (layer F.SilkS)
       (effects (font (size 1 1) (thickness 0.15)))
@@
   )
   (module MX_Alps_Hybrid:MX-1.5U (layer F.Cu)
-    (at 22.225 326.23125)
+    (at 19.05 107.15625)
     (fp_text reference K_LM2 (at 0 3.175) (layer F.SilkS)
       (effects (font (size 1 1) (thickness 0.15)))
@@
   )
   (module MX_Alps_Hybrid:MX-1.5U (layer F.Cu)
-    (at 279.4 326.23125)
+    (at 276.225 107.15625)
     (fp_text reference K_RM12 (at 0 3.175) (layer F.SilkS)
       (effects (font (size 1 1) (thickness 0.15)))
@@
   )
   (module MX_Alps_Hybrid:MX-1.5U (layer F.Cu)
-    (at 231.775 326.23125)
+    (at 228.6 107.15625)
     (fp_text reference K_RM5 (at 0 3.175) (layer F.SilkS)
       (effects (font (size 1 1) (thickness 0.15)))
@@
   )
   (module MX_Alps_Hybrid:MX-1.25U (layer F.Cu)
-    (at 67.46875 326.23125)
+    (at 64.29375 107.15625)
     (fp_text reference K_LM6 (at 0 3.175) (layer F.SilkS)
       (effects (font (size 1 1) (thickness 0.15)))
@@
   )
   (module MX_Alps_Hybrid:MX-1.25U (layer F.Cu)
-    (at 43.65625 326.23125)
+    (at 40.48125 107.15625)
     (fp_text reference K_LM3 (at 0 3.175) (layer F.SilkS)
       (effects (font (size 1 1) (thickness 0.15)))
@@
   )
   (module MX_Alps_Hybrid:MX-1.25U (layer F.Cu)
-    (at 19.84375 326.23125)
+    (at 16.66875 107.15625)
     (fp_text reference K_LM1 (at 0 3.175) (layer F.SilkS)
       (effects (font (size 1 1) (thickness 0.15)))
@@
   )
   (module MX_Alps_Hybrid:MX-1.25U (layer F.Cu)
-    (at 281.78125 326.23125)
+    (at 278.60625 107.15625)
     (fp_text reference K_RM10 (at 0 3.175) (layer F.SilkS)
       (effects (font (size 1 1) (thickness 0.15)))
@@
   )
   (module MX_Alps_Hybrid:MX-1.25U (layer F.Cu)
-    (at 257.96875 326.23125)
+    (at 254.79375 107.15625)
     (fp_text reference K_RM6 (at 0 3.175) (layer F.SilkS)
       (effects (font (size 1 1) (thickness 0.15)))
@@
   )
   (module MX_Alps_Hybrid:MX-1.25U (layer F.Cu)
-    (at 234.15625 326.23125)
+    (at 230.98125 107.15625)
     (fp_text reference K_RM4 (at 0 3.175) (layer F.SilkS)
       (effects (font (size 1 1) (thickness 0.15)))
@@
   )
   (module MX_Alps_Hybrid:MX-1.25U (layer F.Cu)
-    (at 210.34375 326.23125)
+    (at 207.16875 107.15625)
     (fp_text reference K_RM2 (at 0 3.175) (layer F.SilkS)
       (effects (font (size 1 1) (thickness 0.15)))
@@
   )
   (module MX_Alps_Hybrid:MX-1U (layer F.Cu)
-    (at 207.9625 326.23125)
+    (at 204.7875 107.15625)
     (fp_text reference K_RM1 (at 0 3.175) (layer F.SilkS)
       (effects (font (size 1 1) (thickness 0.15)))
@@
   )
   (module MX_Alps_Hybrid:MX-1U (layer F.Cu)
-    (at 227.0125 326.23125)
+    (at 223.8375 107.15625)
     (fp_text reference K_RM3 (at 0 3.175) (layer F.SilkS)
       (effects (font (size 1 1) (thickness 0.15)))
@@
   )
   (module MX_Alps_Hybrid:MX-1U (layer F.Cu)
-    (at 255.5875 326.23125)
+    (at 252.4125 107.15625)
     (fp_text reference K_RM7 (at 0 3.175) (layer F.SilkS)
       (effects (font (size 1 1) (thickness 0.15)))
@@
   )
   (module MX_Alps_Hybrid:MX-1U (layer F.Cu)
-    (at 246.0625 326.23125)
+    (at 242.8875 107.15625)
     (fp_text reference K_RM8 (at 0 3.175) (layer F.SilkS)
       (effects (font (size 1 1) (thickness 0.15)))
@@
   )
   (module MX_Alps_Hybrid:MX-1U (layer F.Cu)
-    (at 265.1125 326.23125)
+    (at 261.9375 107.15625)
     (fp_text reference K_RM9 (at 0 3.175) (layer F.SilkS)
       (effects (font (size 1 1) (thickness 0.15)))
@@
   )
   (module MX_Alps_Hybrid:MX-1U (layer F.Cu)
-    (at 284.1625 326.23125)
+    (at 280.9875 107.15625)
     (fp_text reference K_RM11 (at 0 3.175) (layer F.SilkS)
       (effects (font (size 1 1) (thickness 0.15)))
@@
   )
   (module MX_Alps_Hybrid:MX-1U (layer F.Cu)
-    (at 46.0375 326.23125)
+    (at 42.8625 107.15625)
     (fp_text reference K_LM4 (at 0 3.175) (layer F.SilkS)
       (effects (font (size 1 1) (thickness 0.15)))
@@
   )
   (module MX_Alps_Hybrid:MX-7U-ReversedStabilizers (layer F.Cu)
-    (at 131.7625 326.23125)
+    (at 128.5875 107.15625)
     (fp_text reference K_SP1 (at 0 3.175) (layer F.SilkS)
       (effects (font (size 1 1) (thickness 0.15)))
@@
   )
   (module MX_Alps_Hybrid:MX-6.25U-ReversedStabilizers (layer F.Cu)
-    (at 138.90625 326.23125)
+    (at 135.73125 107.15625)
     (fp_text reference K_SP2 (at 0 3.175) (layer F.SilkS)
       (effects (font (size 1 1) (thickness 0.15)))
@@
   )
   (module MX_Alps_Hybrid:MX-7U-ReversedStabilizers (layer F.Cu)
-    (at 150.8125 326.23125)
+    (at 147.6375 107.15625)
     (fp_text reference K_SP3 (at 0 3.175) (layer F.SilkS)
       (effects (font (size 1 1) (thickness 0.15)))
@@
   )
   (module MX_Alps_Hybrid:MX-6U-7UOverlay (layer F.Cu)
-    (at 141.2875 326.23125)
+    (at 138.1125 107.15625)
     (fp_text reference K_SP3_Extra1 (at 9.525 3.175) (layer F.SilkS)
       (effects (font (size 1 1) (thickness 0.15)))

Commit message: Stack shift row
Parts:
- moved K_RS2 138.1 mm to (235.7, 88.1)
- moved K_RS9 133.6 mm to (271.5, 88.1)
- moved K_RS8 75.3 mm to (273.8, 88.1)
- moved K_RS3 75.3 mm to (245.3, 88.1)
- moved K_LS3 64.1 mm to (14.3, 88.1)
- moved K_LS4 64.1 mm to (33.3, 88.1)
- moved K_RS5 59.5 mm to (254.8, 88.1)
- moved K_LS5 47.6 mm to (16.7, 88.1)
- moved K_LS6 47.6 mm to (38.1, 88.1)
- moved K_,2 42.9 mm to (185.7, 88.1)
- moved K_.2 42.9 mm to (204.8, 88.1)
- moved K_?2 42.9 mm to (223.8, 88.1)
- moved K_B2 42.9 mm to (128.6, 88.1)
- moved K_C2 42.9 mm to (90.5, 88.1)
- moved K_LS2 42.9 mm to (23.8, 88.1)
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Changed lines of the file:
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@@
   )
   (module MX_Alps_Hybrid:MX-2U (layer F.Cu)
-    (at 397.98625 130.96875)
+    (at 271.4625 88.10625)
     (fp_text reference K_RS9 (at 0 3.175) (layer F.SilkS)
       (effects (font (size 1 1) (thickness 0.15)))
@@
   )
   (module MX_Alps_Hybrid:MX-2U (layer F.Cu)
-    (at 23.8125 130.96875)
+    (at 23.8125 88.10625)
     (fp_text reference K_LS2 (at 0 3.175) (layer F.SilkS)
       (effects (font (size 1 1) (thickness 0.15)))
@@
   )
   (module MX_Alps_Hybrid:MX-1.25U (layer F.Cu)
-    (at 307.18125 130.96875)
+    (at 245.26875 88.10625)
     (fp_text reference K_RS3 (at 0 3.175) (layer F.SilkS)
       (effects (font (size 1 1) (thickness 0.15)))
@@
   )
   (module MX_Alps_Hybrid:MX-1.25U (layer F.Cu)
-    (at -30.95625 88.10625)
+    (at 16.66875 88.10625)
     (fp_text reference K_LS5 (at 0 3.175) (layer F.SilkS)
       (effects (font (size 1 1) (thickness 0.15)))
@@
   )
   (module MX_Alps_Hybrid:MX-1U (layer F.Cu)
-    (at 185.7375 130.96875)
+    (at 185.7375 88.10625)
     (fp_text reference K_,2 (at 0 3.175) (layer F.SilkS)
       (effects (font (size 1 1) (thickness 0.15)))
@@
   )
   (module MX_Alps_Hybrid:MX-1U (layer F.Cu)
-    (at 204.7875 130.96875)
+    (at 204.7875 88.10625)
     (fp_text reference K_.2 (at 0 3.175) (layer F.SilkS)
       (effects (font (size 1 1) (thickness 0.15)))
@@
   )
   (module MX_Alps_Hybrid:MX-1U (layer F.Cu)
-    (at 128.5875 130.96875)
+    (at 128.5875 88.10625)
     (fp_text reference K_B2 (at 0 3.175) (layer F.SilkS)
       (effects (font (size 1 1) (thickness 0.15)))
@@
   )
   (module MX_Alps_Hybrid:MX-1U (layer F.Cu)
-    (at 90.4875 130.96875)
+    (at 90.4875 88.10625)
     (fp_text reference K_C2 (at 0 3.175) (layer F.SilkS)
       (effects (font (size 1 1) (thickness 0.15)))
@@
   )
   (module MX_Alps_Hybrid:MX-1U (layer F.Cu)
-    (at -33.3375 130.96875)
+    (at 14.2875 88.10625)
     (fp_text reference K_LS3 (at 0 3.175) (layer F.SilkS)
       (effects (font (size 1 1) (thickness 0.15)))
@@
   )
   (module MX_Alps_Hybrid:MX-1U (layer F.Cu)
-    (at -14.2875 130.96875)
+    (at 33.3375 88.10625)
     (fp_text reference K_LS4 (at 0 3.175) (layer F.SilkS)
       (effects (font (size 1 1) (thickness 0.15)))
@@
   )
   (module MX_Alps_Hybrid:MX-1U (layer F.Cu)
-    (at -9.525 88.10625)
+    (at 38.1 88.10625)
     (fp_text reference K_LS6 (at 0 3.175) (layer F.SilkS)
       (effects (font (size 1 1) (thickness 0.15)))
@@
   )
   (module MX_Alps_Hybrid:MX-1U (layer F.Cu)
-    (at 166.6875 130.96875)
+    (at 166.6875 88.10625)
     (fp_text reference K_M2 (at 0 3.175) (layer F.SilkS)
       (effects (font (size 1 1) (thickness 0.15)))
@@
   )
   (module MX_Alps_Hybrid:MX-1U (layer F.Cu)
-    (at 147.6375 130.96875)
+    (at 147.6375 88.10625)
     (fp_text reference K_N2 (at 0 3.175) (layer F.SilkS)
       (effects (font (size 1 1) (thickness 0.15)))
@@
   )
   (module MX_Alps_Hybrid:MX-1U (layer F.Cu)
-    (at 242.8875 130.96875)
+    (at 242.8875 88.10625)
     (fp_text reference K_RS1 (at 0 3.175) (layer F.SilkS)
       (effects (font (size 1 1) (thickness 0.15)))
@@
   )
   (module MX_Alps_Hybrid:MX-1U (layer F.Cu)
-    (at 261.9375 130.96875)
+    (at 261.9375 88.10625)
     (fp_text reference K_RS4 (at 0 3.175) (layer F.SilkS)
       (effects (font (size 1 1) (thickness 0.15)))
@@
   )
   (module MX_Alps_Hybrid:MX-1U (layer F.Cu)
-    (at 280.9875 130.96875)
+    (at 280.9875 88.10625)
     (fp_text reference K_RS7 (at 0 3.175) (layer F.SilkS)
       (effects (font (size 1 1) (thickness 0.15)))
@@
   )
   (module MX_Alps_Hybrid:MX-1U (layer F.Cu)
-    (at 109.5375 130.96875)
+    (at 109.5375 88.10625)
     (fp_text reference K_V2 (at 0 3.175) (layer F.SilkS)
       (effects (font (size 1 1) (thickness 0.15)))
@@
   )
   (module MX_Alps_Hybrid:MX-1U (layer F.Cu)
-    (at 71.4375 130.96875)
+    (at 71.4375 88.10625)
     (fp_text reference K_X2 (at 0 3.175) (layer F.SilkS)
       (effects (font (size 1 1) (thickness 0.15)))
@@
   )
   (module MX_Alps_Hybrid:MX-1U (layer F.Cu)
-    (at 52.3875 130.96875)
+    (at 52.3875 88.10625)
     (fp_text reference K_Z2 (at 0 3.175) (layer F.SilkS)
       (effects (font (size 1 1) (thickness 0.15)))
@@
   )
   (module MX_Alps_Hybrid:MX-1U (layer F.Cu)
-    (at 223.8375 130.96875)
+    (at 223.8375 88.10625)
     (fp_text reference K_?2 (at 0 3.175) (layer F.SilkS)
       (effects (font (size 1 1) (thickness 0.15)))
@@
   )
   (module MX_Alps_Hybrid:MX-1.75U (layer F.Cu)
-    (at 373.85625 88.10625)
+    (at 235.74375 88.10625)
     (fp_text reference K_RS2 (at 0 3.175) (layer F.SilkS)
       (effects (font (size 1 1) (thickness 0.15)))
@@
   )
   (module MX_Alps_Hybrid:MX-1.75U (layer F.Cu)
-    (at 335.75625 130.96875)
+    (at 273.84375 88.10625)
     (fp_text reference K_RS8 (at 0 3.175) (layer F.SilkS)
       (effects (font (size 1 1) (thickness 0.15)))
@@
   )
   (module MX_Alps_Hybrid:MX-1.75U (layer F.Cu)
-    (at 314.325 88.10625)
+    (at 254.79375 88.10625)
     (fp_text reference K_RS5 (at 0 3.175) (layer F.SilkS)
       (effects (font (size 1 1) (thickness 0.15)))

Commit message: Label excluded keys for prioritization
Other:
- board text added: "Addons to RM7 and RM12"
- board text added: "HHKB Layout"
- board text added: "Orphaned 1U (Perhaps a 2.25U existed to its left before)"
- board text added: "Split 6 Combined with Split 6.25 Var1"
- board text added: "Split 6.25 Variant 1"
- board text added: "Split 6.25 Variant 2"
- board text added: "To left and right: 1.5-1.25-1.5 setups for apple row (6.5U Space shares SP3)"
- board text removed: "RS1 already covered"
- board text removed: "RS4 already covered"
- board text removed: "RS7 already covered"
Changed lines of the file:
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@@
     (area 0 0 0 0)
     (thickness 1.6)
-    (drawings 4)
+    (drawings 7)
     (tracks 278)
     (zones 0)
@@
     (pad "" np_thru_hole circle (at 47.625 -8.255) (size 3.9878 3.9878) (drill 3.9878) (layers *.Cu *.Mask))
   )
-  (gr_text "RS7 already\ncovered" (at 416.71875 88.10625) (layer Dwgs.User)
+  (gr_text "To left and right:\n1.5-1.25-1.5 setups for\napple row (6.5U Space shares SP3)\n" (at 143.66875 285.75) (layer Dwgs.User)
     (effects (font (size 1.5 1.5) (thickness 0.3)))
   )
-  (gr_text "RS4 already\ncovered" (at 400.05 88.10625) (layer Dwgs.User)
+  (gr_text "Addons to\nRM7 and RM12" (at 256.38125 246.85625) (layer Dwgs.User)
     (effects (font (size 1.5 1.5) (thickness 0.3)))
   )
-  (gr_text "RS1 already\ncovered\n" (at 369.09375 130.96875) (layer Dwgs.User)
+  (gr_text "Orphaned 1U\n(Perhaps a 2.25U existed\nto its left before)\n" (at 160.3375 247.65) (layer Dwgs.User)
     (effects (font (size 1.5 1.5) (thickness 0.3)))
   )
-  (gr_text "RS7 already\ncovered" (at 340.51875 88.10625) (layer Dwgs.User)
+  (gr_text "Split 6\nCombined with\nSplit 6.25 Var1" (at 162.71875 228.6) (layer Dwgs.User)
+    (effects (font (size 1.5 1.5) (thickness 0.3)))
+  )
+  (gr_text "Split 6.25\nVariant 2\n" (at 204.7875 190.5 360) (layer Dwgs.User)
+    (effects (font (size 1.5 1.5) (thickness 0.3)))
+  )
+  (gr_text "Split 6.25\nVariant 1" (at 204.7875 170.65625) (layer Dwgs.User)
+    (effects (font (size 1.5 1.5) (thickness 0.3)))
+  )
+  (gr_text "HHKB\nLayout" (at 255.5875 149.225) (layer Dwgs.User)
     (effects (font (size 1.5 1.5) (thickness 0.3)))
   )
